File: cad/elec/giant_midi_keyboard.sch (KiCad schematic (older format))
At the start: 15 parts, among them P1 LEFT, P2 RIGHT, U1 MCP3008, U2 MCP3008, U3 MCP3008, U4 MCP3008, U5 ARDUINO_MICRO

Commit message: Draws first draft of schematics and layout.
Parts:
- added D1, D2, D3, D4: LED, LEDs:LED-5MM, symbol LED
- added R1, R2, R3, R4: 100, Resistors_ThroughHole:Resistor_Horizontal_RM10mm, symbol R
- added R5, R6, R7, R8: 10k, Resistors_ThroughHole:Resistor_Horizontal_RM10mm, symbol R
- U5: footprint (none) -> Giant_Midi_Keyboard:ARDUINO_MICRO
Connections:
- net +5V: now also C3.1, U4.15 (VREF), U4.16 (VDD), R5.1, R6.1, R7.1, R8.1
- net GND: now also U3.9 (DGND), D1.2 (K), D2.2 (K), D3.2 (K), D4.2 (K)
- net L0: now reaches P1.25 (P25), U1.1 (CH0)
- net L0: now also RR1.2; no longer RR1.9
- net CS0: now reaches U1.10 (~CS~/SHDN), U5.4 (0/RX)
- net CS0: now also R5.2
- net SPI_MOSI: now reaches U1.11 (DIN), U2.11 (DIN), U3.11 (DIN), U4.11 (DIN), U5.1 (MOSI)
- net SPI_MISO: now reaches U1.12 (DOUT), U2.12 (DOUT), U3.12 (DOUT), U4.12 (DOUT), U5.33 (MISO)
- net SPI_CLK: now reaches U1.13 (CLK), U2.13 (CLK), U3.13 (CLK), U4.13 (CLK), U5.34 (SCK)
- net L1: now reaches P1.23 (P23), U1.2 (CH1)
- net L1: now also RR1.3; no longer RR1.8
- net L2: now reaches P1.21 (P21), U1.3 (CH2)
- net L2: now also RR1.4; no longer RR1.7
- net L3: now reaches P1.19 (P19), U1.4 (CH3)
- net L3: now also RR1.5; no longer RR1.6
- net L4: now reaches P1.17 (P17), U1.5 (CH4)
- net L4: now also RR1.6; no longer RR1.5
- net L5: now reaches P1.15 (P15), U1.6 (CH5)
- net L5: now also RR1.7; no longer RR1.4
- net L6: now reaches P1.13 (P13), U1.7 (CH6)
- net L6: now also RR1.8; no longer RR1.3
- net L7: now reaches P1.11 (P11), U1.8 (CH7)
- net L7: now also RR1.9; no longer RR1.2
- net L8: now reaches P1.9 (P9), RR2.9
- net L8: now also U2.8 (CH7); no longer U2.1 (CH0)
- net at U5.3 (1/TX): no longer U2.10 (~CS~/SHDN)
- net L9: now reaches P1.7 (P7), RR2.8
- net L9: now also U2.7 (CH6); no longer U2.2 (CH1)
- net L10: now reaches P1.5 (P5), RR2.7
- net L10: now also U2.6 (CH5); no longer U2.3 (CH2)
- net L11: now reaches P1.3 (P3), RR2.6
- net L11: now also U2.5 (CH4); no longer U2.4 (CH3)
- net L12: now reaches P1.1 (P1), RR2.5
- net L12: now also U2.4 (CH3); no longer U2.5 (CH4)
- net L13: now reaches RR2.4
- net L13: now also U2.3 (CH2); no longer U2.6 (CH5)
- net L14: now reaches RR2.3
- net L14: now also U2.2 (CH1); no longer U2.7 (CH6)
- net L15: now reaches RR2.2
- net L15: now also U2.1 (CH0); no longer U2.8 (CH7)
- net R0: now reaches P2.25 (P25), U3.1 (CH0)
- net R0: now also RR3.2; no longer RR3.9
- net CS1: now reaches U5.7 (2/SDA)
- net CS1: now also U2.10 (~CS~/SHDN), R8.2; no longer U3.10 (~CS~/SHDN)
- net R1: now reaches P2.23 (P23), U3.2 (CH1)
- net R1: now also RR3.3; no longer RR3.8
- net R2: now reaches P2.21 (P21), U3.3 (CH2)
- net R2: now also RR3.4; no longer RR3.7
- net R3: now reaches P2.19 (P19), U3.4 (CH3)
- net R3: now also RR3.5; no longer RR3.6
- net R4: now reaches P2.17 (P17), U3.5 (CH4)
- net R4: now also RR3.6; no longer RR3.5
- net R5: now reaches P2.15 (P15), U3.6 (CH5)
- net R5: now also RR3.7; no longer RR3.4
- net R6: now reaches P2.13 (P13), U3.7 (CH6)
- net R6: now also RR3.8; no longer RR3.3
- net R7: now reaches P2.11 (P11), U3.8 (CH7)
- net R7: now also RR3.9; no longer RR3.2
- net R8: now reaches P2.9 (P9), RR4.9
- net R8: now also U4.8 (CH7); no longer U4.1 (CH0)
- net at U5.8 (3(PWM)/SCL): no longer U4.10 (~CS~/SHDN)
- net R9: now reaches P2.7 (P7), RR4.8
- net R9: now also U4.7 (CH6); no longer U4.2 (CH1)
- net R10: now reaches P2.5 (P5), RR4.7
- net R10: now also U4.6 (CH5); no longer U4.3 (CH2)
- net R11: now reaches P2.3 (P3), RR4.6
- net R11: now also U4.5 (CH4); no longer U4.4 (CH3)
- net R12: now reaches P2.1 (P1), RR4.5
- net R12: now also U4.4 (CH3); no longer U4.5 (CH4)
- net R13: now reaches RR4.4
- net R13: now also U4.3 (CH2); no longer U4.6 (CH5)
- net R14: now reaches RR4.3
- net R14: now also U4.2 (CH1); no longer U4.7 (CH6)
- net R15: now reaches RR4.2
- net R15: now also U4.1 (CH0); no longer U4.8 (CH7)
- net CS3: now reaches U5.16 (11(PWM))
- net CS3: now also U4.10 (~CS~/SHDN), R7.2
- net CS2: now reaches U5.17 (12/A11)
- net CS2: now also U3.10 (~CS~/SHDN), R6.2
- net DBG3: now reaches U5.21 (A0)
- net DBG3: now also R4.1
- net DBG2: now reaches U5.22 (A1)
- net DBG2: now also R3.1
- net DBG1: now reaches U5.23 (A2)
- net DBG1: now also R2.1
- net DBG0: now reaches U5.24 (A3)
- net DBG0: now also R1.1
- new net: D2.1 (A), R2.2
- new net: D1.1 (A), R1.2
- new net: D3.1 (A), R3.2
- new net: D4.1 (A), R4.2
Other:
- moved on the sheet: P2, RR1, RR2, RR3, RR4
