File: cad/elec/USB-controller/giant_midi_keyboard.sch (KiCad schematic (older format))
At the start: 27 parts, among them P1 LEFT, P2 RIGHT, U1 MCP3008, U2 MCP3008, U3 MCP3008, U4 MCP3008, U5 ARDUINO_MICRO

Commit message: Updates usb board for use with panel board
Parts:
- removed D1, D2, D3, D4: LED, LEDs:LED-5MM, symbol LED
- removed R1, R2, R3, R4: 100, Resistors_ThroughHole:Resistor_Horizontal_RM10mm, symbol R
- added P3: CONN_01X10, Giant_Midi_Keyboard:Header_2x5, symbol CONN_01X10
- P1, P2: footprint Pin_Headers:Pin_Header_Straight_2x13 -> Giant_Midi_Keyboard:Header_2x13; Part Number T816126A1S101CEU -> T821126A1S100CEU
Connections:
- net +5V: now also P3.10 (P10)
- net GND: now also P3.1 (P1)
- net DBG_I1: now reaches U5.12 (7)
- net DBG_I1: now also P3.8 (P8)
- net DBG_O0: now reaches U5.13 (8/A8)
- net DBG_O0: now also P3.6 (P6)
- net DBG_O2: now reaches U5.14 (9(PWM)/A9)
- net DBG_O2: now also P3.4 (P4)
- net DBG_O4: now reaches U5.15 (10(PWM)/A10)
- net DBG_O4: now also P3.2 (P2)
- net DBG_I2: now reaches U5.25 (A4)
- net DBG_I2: now also P3.7 (P7)
- net DBG_I0: now reaches U5.26 (A5)
- net DBG_I0: now also P3.9 (P9)
- net DBG0 renamed DBG_O1
- net DBG_O1: now also P3.5 (P5)
- net DBG1 renamed DBG_O3
- net DBG_O3: now also P3.3 (P3)
- net DBG2: no longer names the net of U5.22 (A1)
- net DBG3: no longer names the net of U5.21 (A0)
