File: cad/elec/front-panel/front-panel.sch (KiCad schematic (older format))
At the start: 17 parts, among them P1 CONN_01X10, U1 FSM2JAH, U2 FSM2JAH, U3 FSM2JAH

Commit message: Makes the board ready for manual engraving
Parts:
- D1, D2, D3, D4, D5: footprint LEDs:LED-5MM -> Giant Midi Keyboard:LED-5MM
- P1: footprint Socket_Strips:Socket_Strip_Straight_2x05 -> Giant Midi Keyboard:Header_2x5
Changed lines of the file:
@@
 F 0 "P1" H 1050 2300 50  0000 C CNN
 F 1 "CONN_01X10" V 1150 1750 50  0000 C CNN
-F 2 "Socket_Strips:Socket_Strip_Straight_2x05" H 1050 1750 60  0001 C CNN
+F 2 "Giant Midi Keyboard:Header_2x5" H 1050 1750 60  0001 C CNN
 F 3 "" H 1050 1750 60  0000 C CNN
 	1    1050 1750
@@
 F 0 "D1" H 3850 4300 50  0000 C CNN
 F 1 "LED" H 3850 4100 50  0000 C CNN
-F 2 "LEDs:LED-5MM" H 3850 4200 60  0001 C CNN
+F 2 "Giant Midi Keyboard:LED-5MM" H 3850 4200 60  0001 C CNN
 F 3 "" H 3850 4200 60  0000 C CNN
 F 4 "LC503FBL1-15Q-A3-00001 " H 3850 4200 60  0001 C CNN "Part Number"
@@
 F 0 "D2" H 3850 4650 50  0000 C CNN
 F 1 "LED" H 3850 4450 50  0000 C CNN
-F 2 "LEDs:LED-5MM" H 3850 4550 60  0001 C CNN
+F 2 "Giant Midi Keyboard:LED-5MM" H 3850 4550 60  0001 C CNN
 F 3 "" H 3850 4550 60  0000 C CNN
 F 4 "LC503FBL1-15Q-A3-00001 " H 3850 4550 60  0001 C CNN "Part Number"
@@
 F 0 "D3" H 3850 4950 50  0000 C CNN
 F 1 "LED" H 3850 4750 50  0000 C CNN
-F 2 "LEDs:LED-5MM" H 3850 4850 60  0001 C CNN
+F 2 "Giant Midi Keyboard:LED-5MM" H 3850 4850 60  0001 C CNN
 F 3 "" H 3850 4850 60  0000 C CNN
 F 4 "LC503FBL1-15Q-A3-00001 " H 3850 4850 60  0001 C CNN "Part Number"
@@
 F 0 "D4" H 3850 5250 50  0000 C CNN
 F 1 "LED" H 3850 5050 50  0000 C CNN
-F 2 "LEDs:LED-5MM" H 3850 5150 60  0001 C CNN
+F 2 "Giant Midi Keyboard:LED-5MM" H 3850 5150 60  0001 C CNN
 F 3 "" H 3850 5150 60  0000 C CNN
 F 4 "LC503FBL1-15Q-A3-00001 " H 3850 5150 60  0001 C CNN "Part Number"
@@
 F 0 "D5" H 3850 5550 50  0000 C CNN
 F 1 "LED" H 3850 5350 50  0000 C CNN
-F 2 "LEDs:LED-5MM" H 3850 5450 60  0001 C CNN
+F 2 "Giant Midi Keyboard:LED-5MM" H 3850 5450 60  0001 C CNN
 F 3 "" H 3850 5450 60  0000 C CNN
 F 4 "LC503FBL1-15Q-A3-00001 " H 3850 5450 60  0001 C CNN "Part Number"
